File: alpha_pro_micro.kicad_pcb (KiCad board)
At the start: 2 copper layers, 192.9 x 59.5 mm, 62 parts, among them J1 Conn_01x03, K1 KEYSW, K10 KEYSW, K11 KEYSW, K12 KEYSW, K13 KEYSW, K14 KEYSW, K15 KEYSW, K16 KEYSW, K17 KEYSW, K18 KEYSW, K19 KEYSW, K2 KEYSW, K20 KEYSW, K21 KEYSW, K22 KEYSW, K23 KEYSW, K24 KEYSW, K25 KEYSW, K26 KEYSW, K27 KEYSW, K28 KEYSW, K29 KEYSW, K3 KEYSW, K4 KEYSW, K5 KEYSW, K6 KEYSW, K7 KEYSW, K8 KEYSW, K9 KEYSW, SW1 SW_Push, U1 ProMicro

Commit message: footprints, routing
Parts:
- removed SW1: SW_Push, random-keyboard-parts:SKQG-1155865
- removed U1: ProMicro, promicro:ProMicro
- K1, K10, K11, K12, K13, K14, K15, K16, K17, K18, K19, K2, K20, K21, K22, K23, K24, K26, K27, K28, K3, K4, K5, K6, K7, K8, K9: footprint keebio-parts:MX-Alps-Choc-1U-NoLED -> MX_Alps_Hybrid:MXOnly-1U-NoLED
- K25: footprint keebio-parts:MX-Alps-Choc-2U-StabFlip -> MX_Alps_Hybrid:MXOnly-2U-ReversedStabilizers-NoLED
- K29: footprint Keebio-Parts:MX-Alps-Choc-1U-NoLED -> MX_Alps_Hybrid:MXOnly-1U-NoLED
- RZ1: moved to B.Cu
- moved RZ1 17.4 mm to (88.9, 119.7), turned to -90 degrees
- moved D16 3.11 mm to (179.4, 130.2)
- moved D28 0.13 mm to (236.5, 149.2)
- moved D10 0.06 mm to (255.6, 111.1)
- moved D29 0.06 mm to (255.6, 149.2)
- moved D6 0.06 mm to (179.4, 111.2)
- moved D7 0.06 mm to (198.4, 111.1)
- moved D8 0.06 mm to (217.5, 111.1)
- moved D9 0.06 mm to (236.5, 111.2)
Connections:
- D25 pad 2: Net-(D25-Pad2) -> Net-(K25-Pad1)
- K25 pad 1: /col5 -> Net-(K25-Pad1)
- K25 pad 2: Net-(D25-Pad2) -> /col5
Routing:
- net /row2: track 349.8 -> 0.00 mm
- net /row0: track 340.9 -> 0.00 mm
- net /row1: track 326.7 -> 0.00 mm
- net /col2: track 71.7 -> 0.00 mm
- net /col0: track 56.3 -> 0.00 mm
- net /col1: track 55.3 -> 0.00 mm, vias 1 -> 0
- net /col5: track 51.2 -> 0.00 mm
- net /col9: track 50.5 -> 0.00 mm
- net /col8: track 50.4 -> 0.00 mm
- net /col3: track 50.4 -> 0.00 mm
- net /col6: track 50.4 -> 0.00 mm
- net /col7: track 50.4 -> 0.00 mm
- net /col4: track 27.8 -> 0.00 mm
- net Net-(D11-Pad2): track 22.5 -> 0.00 mm
- net Net-(D16-Pad2): track 10.0 -> 0.00 mm
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Other:
- board size 192.9 x 59.5 mm -> 192.9 x 55 mm
- board text added: "bumpon feet where?"
- board text added: "swap controller footprint to bottom?"
