File: alpha_pro_micro.kicad_sch (KiCad schematic)
At the start: 62 parts, among them J1 Conn_01x03, K1 KEYSW, K10 KEYSW, K11 KEYSW, K12 KEYSW, K13 KEYSW, K14 KEYSW, K15 KEYSW, K16 KEYSW, K17 KEYSW, K18 KEYSW, K19 KEYSW, K2 KEYSW, K20 KEYSW, K21 KEYSW, K22 KEYSW, K23 KEYSW, K24 KEYSW, K25 KEYSW, K26 KEYSW, K27 KEYSW, K28 KEYSW, K29 KEYSW, K3 KEYSW, K4 KEYSW, K5 KEYSW, K6 KEYSW, K7 KEYSW, K8 KEYSW, K9 KEYSW, SW1 SW_Push, U1 ProMicro

Commit message: footprints, routing
Parts:
- removed SW1: SW_Push, random-keyboard-parts:SKQG-1155865, symbol Switch:SW_Push
- removed U1: ProMicro, promicro:ProMicro, symbol alpha_pro_micro-rescue:ProMicro
- K1, K10, K11, K12, K13, K14, K15, K16, K17, K18, K19, K2, K20, K21, K22, K23, K24, K26, K27, K28, K3, K4, K5, K6, K7, K8, K9: footprint keebio-parts:MX-Alps-Choc-1U-NoLED -> MX_Alps_Hybrid:MXOnly-1U-NoLED
- K25: footprint keebio-parts:MX-Alps-Choc-2U-StabFlip -> MX_Alps_Hybrid:MXOnly-2U-ReversedStabilizers-NoLED
- K29: footprint Keebio-Parts:MX-Alps-Choc-1U-NoLED -> MX_Alps_Hybrid:MXOnly-1U-NoLED
Connections:
- net col5: now also K25.2; no longer K25.1
- net at D25.2 (A): now also K25.1; no longer K25.2
Other:
- moved on the sheet: J1, K25

Commit message: alpha29 completed, but untested
Connections:
- net VCC is gone; now on net +5V: J1.1 (Pin_1)
- net RGB: now also RZ1.20 (GP29); no longer RZ1.14 (GP13)
- net col0: now also RZ1.5 (GP4); no longer RZ1.19 (GP28)
- net col1: now also RZ1.13 (GP12); no longer RZ1.18 (GP27)
- net col2: now also RZ1.7 (GP6); no longer RZ1.17 (GP26)
- net col3: now also RZ1.14 (GP13); no longer RZ1.16 (GP15)
- net col4: now also RZ1.15 (GP14); no longer RZ1.8 (GP7)
- net col5: now also RZ1.8 (GP7); no longer RZ1.7 (GP6)
- net col6: now also RZ1.16 (GP15); no longer RZ1.6 (GP5)
- net col7: now also RZ1.9 (GP8); no longer RZ1.5 (GP4)
- net col8: now also RZ1.17 (GP26); no longer RZ1.4 (GP3)
- net col9: now also RZ1.10 (GP9); no longer RZ1.3 (GP2)
- net row0: now also RZ1.18 (GP27); no longer RZ1.10 (GP9)
- net row1: now also RZ1.11 (GP10); no longer RZ1.15 (GP14)
- net row2: now also RZ1.6 (GP5); no longer RZ1.20 (GP29)
Other:
- note added: "is +5V okaz instead of VVC?"
- note added: "what is that?"
Changed lines of the file:
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@@
     (stroke (width 0) (type default) (color 0 0 0 0))
   )
-  (label "col7" (at 46.99 50.165 180)
+  (text "is +5V okaz instead of VVC?" (at 104.775 34.29 0)
+    (effects (font (size 1.27 1.27)) (justify left bottom))
+  )
+  (text "what is that?\n" (at 92.075 26.67 0)
+    (effects (font (size 1.27 1.27)) (justify left bottom))
+  )
+  (label "col7" (at 46.99 60.325 180)
     (effects (font (size 1.524 1.524)) (justify right bottom))
   )
-  (label "col6" (at 46.99 52.705 180)
-    (effects (font (size 1.524 1.524)) (justify right bottom))
-  )
-  (label "row1" (at 76.2 52.705 0)
+  (label "col6" (at 76.2 50.165 0)
+    (effects (font (size 1.524 1.524)) (justify left bottom))
+  )
+  (label "row1" (at 76.2 62.865 0)
     (effects (font (size 1.524 1.524)) (justify left bottom))
   )
@@
     (effects (font (size 1.524 1.524)) (justify left bottom))
   )
-  (label "col0" (at 76.2 42.545 0)
-    (effects (font (size 1.524 1.524)) (justify left bottom))
-  )
-  (label "row2" (at 76.2 40.005 0)
-    (effects (font (size 1.524 1.524)) (justify left bottom))
-  )
-  (label "col8" (at 46.99 47.625 180)
+  (label "col0" (at 46.99 50.165 180)
     (effects (font (size 1.524 1.524)) (justify right bottom))
   )
+  (label "row2" (at 46.99 52.705 180)
+    (effects (font (size 1.524 1.524)) (justify right bottom))
+  )
+  (label "col8" (at 76.2 47.625 0)
+    (effects (font (size 1.524 1.524)) (justify left bottom))
+  )
   (label "col0" (at 40.64 91.44 90)
     (effects (font (size 1.524 1.524)) (justify left bottom))
@@
     (effects (font (size 1.524 1.524)) (justify left bottom))
   )
-  (label "row0" (at 46.99 62.865 180)
+  (label "row0" (at 76.2 45.085 0)
+    (effects (font (size 1.524 1.524)) (justify left bottom))
+  )
+  (label "col4" (at 139.7 90.17 90)
+    (effects (font (size 1.524 1.524)) (justify left bottom))
+  )
+  (label "col1" (at 76.2 57.785 0)
+    (effects (font (size 1.524 1.524)) (justify left bottom))
+  )
+  (label "col9" (at 46.99 62.865 180)
     (effects (font (size 1.524 1.524)) (justify right bottom))
   )
-  (label "col4" (at 139.7 90.17 90)
-    (effects (font (size 1.524 1.524)) (justify left bottom))
-  )
-  (label "col1" (at 76.2 45.085 0)
-    (effects (font (size 1.524 1.524)) (justify left bottom))
-  )
-  (label "col9" (at 46.99 45.085 180)
+  (label "col8" (at 241.3 91.44 90)
+    (effects (font (size 1.524 1.524)) (justify left bottom))
+  )
+  (label "col5" (at 46.99 57.785 180)
     (effects (font (size 1.524 1.524)) (justify right bottom))
   )
-  (label "col8" (at 241.3 91.44 90)
-    (effects (font (size 1.524 1.524)) (justify left bottom))
-  )
-  (label "col5" (at 46.99 55.245 180)
-    (effects (font (size 1.524 1.524)) (justify right bottom))
-  )
-  (label "col4" (at 46.99 57.785 180)
-    (effects (font (size 1.524 1.524)) (justify right bottom))
+  (label "col4" (at 76.2 52.705 0)
+    (effects (font (size 1.524 1.524)) (justify left bottom))
   )
   (label "col6" (at 191.77 91.44 90)
@@
     (effects (font (size 1.524 1.524)) (justify left bottom))
   )
-  (label "col2" (at 76.2 47.625 0)
-    (effects (font (size 1.524 1.524)) (justify left bottom))
-  )
-  (label "col3" (at 76.2 50.165 0)
+  (label "col2" (at 46.99 55.245 180)
+    (effects (font (size 1.524 1.524)) (justify right bottom))
+  )
+  (label "col3" (at 76.2 55.245 0)
     (effects (font (size 1.524 1.524)) (justify left bottom))
   )
@@
     )
   )
-  (global_label "RGB" (shape input) (at 76.2 55.245 0) (fields_autoplaced)
+  (global_label "RGB" (shape input) (at 76.2 40.005 0) (fields_autoplaced)
     (effects (font (size 1.27 1.27)) (justify left))
-    (property "Intersheet References" "${INTERSHEET_REFS}" (id 0) (at -60.96 8.255 0)
+    (property "Intersheet References" "${INTERSHEET_REFS}" (id 0) (at -60.96 -6.985 0)
       (effects (font (size 1.27 1.27)) hide)
     )
@@
     (pin "2")
     (pin "3")
-  )
-  (symbol (lib_id "power:VCC") (at 129.54 37.465 90) (unit 1)
-    (in_bom yes) (on_board yes)
-    (property "Reference" "#PWR05" (id 0) (at 133.35 37.465 0)
-      (effects (font (size 1.27 1.27)) hide)
-    )
-    (property "Value" "VCC" (id 1) (at 125.73 37.465 0))
-    (property "Footprint" "" (id 2) (at 129.54 37.465 0)
-      (effects (font (size 1.27 1.27)) hide)
-    )
-    (property "Datasheet" "" (id 3) (at 129.54 37.465 0)
-      (effects (font (size 1.27 1.27)) hide)
-    )
-    (pin "1")
   )
   (symbol (lib_id "power:GND") (at 129.54 42.545 270) (unit 1)
@@
     (pin "9")
   )
+  (symbol (lib_id "power:+5V") (at 129.54 37.465 90) (unit 1)
+    (in_bom yes) (on_board yes) (fields_autoplaced)
+    (property "Reference" "#PWR0101" (id 0) (at 133.35 37.465 0)
+      (effects (font (size 1.27 1.27)) hide)
+    )
+    (property "Value" "+5V" (id 1) (at 125.73 37.4649 90)
+      (effects (font (size 1.27 1.27)) (justify left))
+    )
+    (property "Footprint" "" (id 2) (at 129.54 37.465 0)
+      (effects (font (size 1.27 1.27)) hide)
+    )
+    (property "Datasheet" "" (id 3) (at 129.54 37.465 0)
+      (effects (font (size 1.27 1.27)) hide)
+    )
+    (pin "1")
+  )
   (sheet_instances
     (path "/" (page "1"))
@@
       (reference "#PWR03") (unit 1) (value "GND") (footprint "")
     )
-    (path "/00000000-0000-0000-0000-00005ab44c2d"
-      (reference "#PWR05") (unit 1) (value "VCC") (footprint "")
-    )
     (path "/00000000-0000-0000-0000-00005ab44d66"
       (reference "#PWR06") (unit 1) (value "GND") (footprint "")
     )
+    (path "/dbd7b615-d46e-47dd-84c8-3e425097e1f8"
+      (reference "#PWR0101") (unit 1) (value "+5V") (footprint "")
+    )
     (path "/36c89016-d05b-45a6-b9c7-d9fda913b705"
