File: Project/alpha_pro_micro.kicad_sch (KiCad schematic)
At the start: 60 parts, among them J1 Conn_01x03, K1 KEYSW, K10 KEYSW, K11 KEYSW, K12 KEYSW, K13 KEYSW, K14 KEYSW, K15 KEYSW, K16 KEYSW, K17 KEYSW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

Commit message: backup
Other:
- note removed: "is +5V okaz instead of VVC?"
- note removed: "what is that?"
Changed lines of the file:
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@@
     (stroke (width 0) (type default) (color 0 0 0 0))
-  )
-  (text "is +5V okaz instead of VVC?" (at 104.775 34.29 0)
-    (effects (font (size 1.27 1.27)) (justify left bottom))
-  )
-  (text "what is that?\n" (at 92.075 26.67 0)
-    (effects (font (size 1.27 1.27)) (justify left bottom))
   )
   (label "col7" (at 46.99 60.325 180)
@@
     (effects (font (size 1.524 1.524)) (justify left bottom))
   )
-  (label "col_tmo" (at 99.06 23.495 180)
-    (effects (font (size 1.27 1.27)) (justify right bottom))
-  )
   (label "row2" (at 16.51 146.05 180)
